Commit message: Rename imu_link to imu

File: mini_pupper_description/urdf/mini_pupper_description.urdf.xacro (robot description, xacro)
@@ -1781,5 +1781,5 @@
     </plugin>
   </gazebo>
-  <link name="imu_link">
+  <link name="imu">
     <inertial>
       <mass value="0.0001"/>
@@ -1790,7 +1790,7 @@
   <joint name="imu_joint" type="fixed">
     <parent link="base_link"/>
-    <child link="imu_link"/>
-  </joint>
-  <gazebo reference="imu_link">
+    <child link="imu"/>
+  </joint>
+  <gazebo reference="imu">
     <sensor name="imu_controller" type="imu">
       <always_on>true</always_on>
